File: MCU.kicad_sch (KiCad schematic)
At the start: 7 parts, among them U2 LAUNCHXL-F28379D

Commit message: new CSV uploaded
Parts:
- D3(Red)1: renamed from D3; Part Number (none) -> LTST-C150KRKT
- D4(green)1: renamed from D4; Part Number (none) -> LTST-C150KGKT
- D5(Blue)1: renamed from D5; Part Number (none) -> LTST-C150TBKT
Changed lines of the file:
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@@
 		(on_board yes)
 		(dnp no)
-		(property "Reference" "D5"
-			(at 66.04 27.94 0)
+		(property "Reference" "D5(Blue)1"
+			(at 60.452 27.686 0)
 			(effects
 				(font
@@
 			)
 		)
-		(property "Datasheet" "http://www.everlight.com/file/ProductFile/IR26-21C-L110-TR8.pdf"
+		(property "Datasheet" "https://optoelectronics.liteon.com/upload/download/DS22-2000-026/LTST-C150TBKT(0630).pdf"
 			(at 67.31 30.48 0)
 			(effects
@@
 		)
 		(property "Description" "940nm, 20 deg, Infrared LED, 1206"
+			(at 67.31 30.48 0)
+			(effects
+				(font
+					(size 1.27 1.27)
+				)
+				(hide yes)
+			)
+		)
+		(property "Part Number" "LTST-C150TBKT"
 			(at 67.31 30.48 0)
 			(effects
@@
 			(project "MyFirstBuck"
 				(path "/0768732b-0e8f-4a40-9cf3-e602ee34def3/93d2fcfa-d06c-41b2-bece-4410c3be6b80"
-					(reference "D5")
+					(reference "D5(Blue)1")
 					(unit 1)
 				)
@@
 		(on_board yes)
 		(dnp no)
-		(property "Reference" "D3"
-			(at 66.04 14.732 0)
+		(property "Reference" "D3(Red)1"
+			(at 62.992 13.97 0)
 			(effects
 				(font
@@
 			)
 		)
-		(property "Datasheet" "http://www.everlight.com/file/ProductFile/IR26-21C-L110-TR8.pdf"
+		(property "Datasheet" "https://optoelectronics.liteon.com/upload/download/DS-22-99-0149/LTST-C150KRKT.pdf"
 			(at 67.31 17.78 0)
 			(effects
@@
 		)
 		(property "Description" "940nm, 20 deg, Infrared LED, 1206"
+			(at 67.31 17.78 0)
+			(effects
+				(font
+					(size 1.27 1.27)
+				)
+				(hide yes)
+			)
+		)
+		(property "Part Number" "LTST-C150KRKT"
 			(at 67.31 17.78 0)
 			(effects
@@
 			(project "MyFirstBuck"
 				(path "/0768732b-0e8f-4a40-9cf3-e602ee34def3/93d2fcfa-d06c-41b2-bece-4410c3be6b80"
-					(reference "D3")
+					(reference "D3(Red)1")
 					(unit 1)
 				)
@@
 		(on_board yes)
 		(dnp no)
-		(property "Reference" "D4"
-			(at 65.786 22.606 0)
+		(property "Reference" "D4(green)1"
+			(at 61.214 22.098 0)
 			(effects
 				(font
@@
 			)
 		)
-		(property "Datasheet" "http://www.everlight.com/file/ProductFile/IR26-21C-L110-TR8.pdf"
+		(property "Datasheet" "https://optoelectronics.liteon.com/upload/download/DS22-2000-072/LTST-C150KGKT.pdf"
 			(at 67.31 25.4 0)
 			(effects
@@
 		)
 		(property "Description" "940nm, 20 deg, Infrared LED, 1206"
+			(at 67.31 25.4 0)
+			(effects
+				(font
+					(size 1.27 1.27)
+				)
+				(hide yes)
+			)
+		)
+		(property "Part Number" "LTST-C150KGKT"
 			(at 67.31 25.4 0)
 			(effects
@@
 			(project "MyFirstBuck"
 				(path "/0768732b-0e8f-4a40-9cf3-e602ee34def3/93d2fcfa-d06c-41b2-bece-4410c3be6b80"
-					(reference "D4")
+					(reference "D4(green)1")
 					(unit 1)
 				)
